Commit message: name the legs after the side they are actually on
The chain called L_ sat at y = -0.1237. Forward is +x -- bending a knee
60 degrees drives the foot 0.41 m along -x, and knees bend backward --
so in a right-handed frame with z up, +y is left and every L_ name was
on the right leg. That has been true since the project's first model on
2026-06-21 and was written into the v2 builder on 2026-08-22.

Inside the simulator it was harmless: a mirrored robot with swapped
labels is the same robot. It only bit when the real legs were wired up
and the left knee got the right knee's limits, so the safety clamp spent
the day pressing that knee into its hard stop.

Swap the prefixes in 67 model files, the two mirrored hip_yaw keyframe
values that go with them, our limit files, and the audit harness. Body
positions, masses, inertias, axes and ranges are byte-identical -- only
names moved, so trained policies still drive the same joints in the same
order. build_robot.py now refuses to write a model whose L_ chain is on
the -y side.

File: pygmalion_locomotion/assets/pygmalion_v2/pygmalion_v2.urdf (robot description, URDF)
Before this commit: robot pygmalion_v2, 18 links, 17 joints
Links:
- removed link L_arm_link
- removed link L_shoulder_pitch_link
- removed link R_arm_link
- removed link R_shoulder_pitch_link
- removed link torso_link
- link L_ankle_pitch_link: mass 0.084987 -> 0.086895
- link L_foot_link: mass 1.0304 -> 0.77534; geometry collision mesh filename=meshes/R_foot_hull.stl; visual mesh filename=meshes/R_foot.stl
- link L_hip_pitch_link: mass 2.1738 -> 2.1779; geometry collision mesh filename=meshes/R_hip_pitch_link_hull.stl; visual mesh filename=meshes/R_hip_pitch_link.stl
- link L_hip_roll_link: mass 1.6181 -> 1.8198; geometry collision mesh filename=meshes/R_hip_roll_link_hull.stl; visual mesh filename=meshes/R_hip_roll_link.stl
- link L_shin_link: mass 3.6275 -> 3.3529; geometry collision mesh filename=meshes/R_shin_hull.stl; visual mesh filename=meshes/R_shin.stl
- link L_thigh_link: mass 2.9294 -> 2.7562; geometry collision mesh filename=meshes/R_thigh_hull.stl; visual mesh filename=meshes/R_thigh.stl
- link R_ankle_pitch_link: mass 0.084987 -> 0.086895
- link R_foot_link: mass 1.0304 -> 0.77534; geometry collision mesh filename=meshes/foot_hull.stl; visual mesh filename=meshes/foot.stl
- link R_hip_pitch_link: mass 2.1738 -> 2.1779; geometry collision mesh filename=meshes/hip_pitch_link_hull.stl; visual mesh filename=meshes/hip_pitch_link.stl
- link R_hip_roll_link: mass 1.6181 -> 1.8198; geometry collision mesh filename=meshes/hip_roll_link_hull.stl; visual mesh filename=meshes/hip_roll_link.stl
- link R_shin_link: mass 3.6275 -> 3.3529; geometry collision mesh filename=meshes/shin_hull.stl; visual mesh filename=meshes/shin.stl
- link R_thigh_link: mass 2.9294 -> 2.7562; geometry collision mesh filename=meshes/thigh_hull.stl; visual mesh filename=meshes/thigh.stl
- link base_link: mass 5.3668 -> 21.763
Joints:
- removed joint L_shoulder_pitch_joint
- removed joint L_shoulder_roll_joint
- removed joint R_shoulder_pitch_joint
- removed joint R_shoulder_roll_joint
- removed joint waist_yaw_joint
- joint L_ankle_roll_joint: axis -1 0 0 -> 1 0 0
- joint L_hip_pitch_joint: origin xyz=0 -0.1237 0 rpy=0 0 0 -> xyz=0 0.1237 0 rpy=0 0 0
- joint L_hip_roll_joint: axis 1 0 0 -> -1 0 0
- joint R_ankle_roll_joint: axis 1 0 0 -> -1 0 0
- joint R_hip_pitch_joint: origin xyz=0 0.1237 0 rpy=0 0 0 -> xyz=0 -0.1237 0 rpy=0 0 0
- joint R_hip_roll_joint: axis -1 0 0 -> 1 0 0

File: pygmalion_locomotion/assets/pygmalion_v2/pygmalion_v3_printed.urdf (robot description, URDF)
Before this commit: robot pygmalion_v3_printed, 18 links, 17 joints
Links:
- link L_arm_link: geometry collision mesh filename=meshes/R_arm_hull.stl; visual mesh filename=meshes/R_arm.stl
- link L_foot_link: geometry collision mesh filename=meshes/R_foot_hull.stl; visual mesh filename=meshes/R_foot.stl
- link L_hip_pitch_link: geometry collision mesh filename=meshes/R_hip_pitch_link_hull.stl; visual mesh filename=meshes/R_hip_pitch_link.stl
- link L_hip_roll_link: geometry collision mesh filename=meshes/R_hip_roll_link_hull.stl; visual mesh filename=meshes/R_hip_roll_link.stl
- link L_shin_link: geometry collision mesh filename=meshes/R_shin_hull.stl; visual mesh filename=meshes/R_shin.stl
- link L_shoulder_pitch_link: geometry collision mesh filename=meshes/R_shoulder_pitch_link_hull.stl; visual mesh filename=meshes/R_shoulder_pitch_link.stl
- link L_thigh_link: geometry collision mesh filename=meshes/R_thigh_hull.stl; visual mesh filename=meshes/R_thigh.stl
- link R_arm_link: geometry collision mesh filename=meshes/arm_hull.stl; visual mesh filename=meshes/arm.stl
- link R_foot_link: geometry collision mesh filename=meshes/foot_hull.stl; visual mesh filename=meshes/foot.stl
- link R_hip_pitch_link: geometry collision mesh filename=meshes/hip_pitch_link_hull.stl; visual mesh filename=meshes/hip_pitch_link.stl
- link R_hip_roll_link: geometry collision mesh filename=meshes/hip_roll_link_hull.stl; visual mesh filename=meshes/hip_roll_link.stl
- link R_shin_link: geometry collision mesh filename=meshes/shin_hull.stl; visual mesh filename=meshes/shin.stl
- link R_shoulder_pitch_link: geometry collision mesh filename=meshes/shoulder_pitch_link_hull.stl; visual mesh filename=meshes/shoulder_pitch_link.stl
- link R_thigh_link: geometry collision mesh filename=meshes/thigh_hull.stl; visual mesh filename=meshes/thigh.stl
Joints:
- joint L_ankle_roll_joint: axis -1 0 0 -> 1 0 0
- joint L_hip_pitch_joint: origin xyz=0 -0.1237 0 rpy=0 0 0 -> xyz=0 0.1237 0 rpy=0 0 0
- joint L_hip_roll_joint: axis 1 0 0 -> -1 0 0
- joint L_shoulder_pitch_joint: origin xyz=-0.015 -0.2 0.3625 rpy=0 0 0 -> xyz=-0.015 0.2 0.3625 rpy=0 0 0
- joint L_shoulder_roll_joint: axis 1 0 0 -> -1 0 0
- joint R_ankle_roll_joint: axis 1 0 0 -> -1 0 0
- joint R_hip_pitch_joint: origin xyz=0 0.1237 0 rpy=0 0 0 -> xyz=0 -0.1237 0 rpy=0 0 0
- joint R_hip_roll_joint: axis -1 0 0 -> 1 0 0
- joint R_shoulder_pitch_joint: origin xyz=-0.015 0.2 0.3625 rpy=0 0 0 -> xyz=-0.015 -0.2 0.3625 rpy=0 0 0
- joint R_shoulder_roll_joint: axis -1 0 0 -> 1 0 0

File: pygmalion_locomotion/assets/pygmalion_v2/pygmalion_v3_printed_loop.urdf (robot description, URDF)
Before this commit: robot pygmalion_v3_printed_loop, 30 links, 29 joints
Links:
- link L_arm_link: geometry collision mesh filename=meshes/R_arm_hull.stl; visual mesh filename=meshes/R_arm.stl
- link L_crank_A: geometry visual mesh filename=meshes/R_crank_A.stl
- link L_crank_B: geometry visual mesh filename=meshes/R_crank_B.stl
- link L_foot_link: geometry collision mesh filename=meshes/R_foot_hull.stl; visual mesh filename=meshes/R_foot.stl
- link L_hip_pitch_link: geometry collision mesh filename=meshes/R_hip_pitch_link_hull.stl; visual mesh filename=meshes/R_hip_pitch_link.stl
- link L_hip_roll_link: geometry collision mesh filename=meshes/R_hip_roll_link_hull.stl; visual mesh filename=meshes/R_hip_roll_link.stl
- link L_rod_A: geometry visual mesh filename=meshes/R_rod_A.stl
- link L_rod_B: geometry visual mesh filename=meshes/R_rod_B.stl
- link L_shin_link: geometry collision mesh filename=meshes/R_shin_hull.stl; visual mesh filename=meshes/R_shin.stl
- link L_shoulder_pitch_link: geometry collision mesh filename=meshes/R_shoulder_pitch_link_hull.stl; visual mesh filename=meshes/R_shoulder_pitch_link.stl
- link L_thigh_link: geometry collision mesh filename=meshes/R_thigh_hull.stl; visual mesh filename=meshes/R_thigh.stl
- link R_arm_link: geometry collision mesh filename=meshes/arm_hull.stl; visual mesh filename=meshes/arm.stl
- link R_crank_A: geometry visual mesh filename=meshes/crank_A.stl
- link R_crank_B: geometry visual mesh filename=meshes/crank_B.stl
- link R_foot_link: geometry collision mesh filename=meshes/foot_hull.stl; visual mesh filename=meshes/foot.stl
- link R_hip_pitch_link: geometry collision mesh filename=meshes/hip_pitch_link_hull.stl; visual mesh filename=meshes/hip_pitch_link.stl
- link R_hip_roll_link: geometry collision mesh filename=meshes/hip_roll_link_hull.stl; visual mesh filename=meshes/hip_roll_link.stl
- link R_rod_A: geometry visual mesh filename=meshes/rod_A.stl
- link R_rod_B: geometry visual mesh filename=meshes/rod_B.stl
- link R_shin_link: geometry collision mesh filename=meshes/shin_hull.stl; visual mesh filename=meshes/shin.stl
- link R_shoulder_pitch_link: geometry collision mesh filename=meshes/shoulder_pitch_link_hull.stl; visual mesh filename=meshes/shoulder_pitch_link.stl
- link R_thigh_link: geometry collision mesh filename=meshes/thigh_hull.stl; visual mesh filename=meshes/thigh.stl
Joints:
- joint L_ankle_roll_joint: axis -1 0 0 -> 1 0 0
- joint L_crank_A_joint: origin xyz=-0.029945 -0.001718 -0.190034 rpy=0 0 0 -> xyz=-0.029945 0.001718 -0.190034 rpy=0 0 0
- joint L_crank_B_joint: origin xyz=-0.030055 0.001717 -0.290034 rpy=0 0 0 -> xyz=-0.030055 -0.001717 -0.290034 rpy=0 0 0
- joint L_hip_pitch_joint: origin xyz=0 -0.1237 0 rpy=0 0 0 -> xyz=0 0.1237 0 rpy=0 0 0
- joint L_hip_roll_joint: axis 1 0 0 -> -1 0 0
- joint L_rod_A_u1: origin xyz=-0.061494 0.042718 -0.021185 rpy=0 0 0 -> xyz=-0.061494 -0.042718 -0.021185 rpy=0 0 0
- joint L_rod_B_u1: origin xyz=-0.060039 -0.042717 -0.01522 rpy=0 0 0 -> xyz=-0.060039 0.042717 -0.01522 rpy=0 0 0
- joint L_shoulder_pitch_joint: origin xyz=-0.015 -0.2 0.3625 rpy=0 0 0 -> xyz=-0.015 0.2 0.3625 rpy=0 0 0
- joint L_shoulder_roll_joint: axis 1 0 0 -> -1 0 0
- joint R_ankle_roll_joint: axis 1 0 0 -> -1 0 0
- joint R_crank_A_joint: origin xyz=-0.029945 0.001718 -0.190034 rpy=0 0 0 -> xyz=-0.029945 -0.001718 -0.190034 rpy=0 0 0
- joint R_crank_B_joint: origin xyz=-0.030055 -0.001717 -0.290034 rpy=0 0 0 -> xyz=-0.030055 0.001717 -0.290034 rpy=0 0 0
- joint R_hip_pitch_joint: origin xyz=0 0.1237 0 rpy=0 0 0 -> xyz=0 -0.1237 0 rpy=0 0 0
- joint R_hip_roll_joint: axis -1 0 0 -> 1 0 0
- joint R_rod_A_u1: origin xyz=-0.061494 -0.042718 -0.021185 rpy=0 0 0 -> xyz=-0.061494 0.042718 -0.021185 rpy=0 0 0
- joint R_rod_B_u1: origin xyz=-0.060039 0.042717 -0.01522 rpy=0 0 0 -> xyz=-0.060039 -0.042717 -0.01522 rpy=0 0 0
- joint R_shoulder_pitch_joint: origin xyz=-0.015 0.2 0.3625 rpy=0 0 0 -> xyz=-0.015 -0.2 0.3625 rpy=0 0 0
- joint R_shoulder_roll_joint: axis -1 0 0 -> 1 0 0

File: pygmalion_locomotion/assets/pygmalion_v2/pygmalion_v4_printed.urdf (robot description, URDF)
Before this commit: robot pygmalion_v4_printed, 18 links, 17 joints
Links:
- link L_arm_link: geometry collision mesh filename=meshes/R_arm_hull.stl; visual mesh filename=meshes/R_arm.stl
- link L_foot_link: geometry collision mesh filename=meshes/R_foot_hull.stl; visual mesh filename=meshes/R_foot.stl
- link L_hip_pitch_link: geometry collision mesh filename=meshes/R_hip_pitch_link_hull.stl; visual mesh filename=meshes/R_hip_pitch_link.stl
- link L_hip_roll_link: geometry collision mesh filename=meshes/R_hip_roll_link_hull.stl; visual mesh filename=meshes/R_hip_roll_link.stl
- link L_shin_link: geometry collision mesh filename=meshes/R_shin_hull.stl; visual mesh filename=meshes/R_shin.stl
- link L_shoulder_pitch_link: geometry collision mesh filename=meshes/R_shoulder_pitch_link_hull.stl; visual mesh filename=meshes/R_shoulder_pitch_link.stl
- link L_thigh_link: geometry collision mesh filename=meshes/R_thigh_hull.stl; visual mesh filename=meshes/R_thigh.stl
- link R_arm_link: geometry collision mesh filename=meshes/arm_hull.stl; visual mesh filename=meshes/arm.stl
- link R_foot_link: geometry collision mesh filename=meshes/foot_hull.stl; visual mesh filename=meshes/foot.stl
- link R_hip_pitch_link: geometry collision mesh filename=meshes/hip_pitch_link_hull.stl; visual mesh filename=meshes/hip_pitch_link.stl
- link R_hip_roll_link: geometry collision mesh filename=meshes/hip_roll_link_hull.stl; visual mesh filename=meshes/hip_roll_link.stl
- link R_shin_link: geometry collision mesh filename=meshes/shin_hull.stl; visual mesh filename=meshes/shin.stl
- link R_shoulder_pitch_link: geometry collision mesh filename=meshes/shoulder_pitch_link_hull.stl; visual mesh filename=meshes/shoulder_pitch_link.stl
- link R_thigh_link: geometry collision mesh filename=meshes/thigh_hull.stl; visual mesh filename=meshes/thigh.stl
Joints:
- joint L_ankle_roll_joint: axis -1 0 0 -> 1 0 0
- joint L_hip_pitch_joint: origin xyz=0 -0.1237 0 rpy=0 0 0 -> xyz=0 0.1237 0 rpy=0 0 0
- joint L_hip_roll_joint: axis 1 0 0 -> -1 0 0
- joint L_shoulder_pitch_joint: origin xyz=-0.015 -0.2 0.3625 rpy=0 0 0 -> xyz=-0.015 0.2 0.3625 rpy=0 0 0
- joint L_shoulder_roll_joint: axis 1 0 0 -> -1 0 0
- joint R_ankle_roll_joint: axis 1 0 0 -> -1 0 0
- joint R_hip_pitch_joint: origin xyz=0 0.1237 0 rpy=0 0 0 -> xyz=0 -0.1237 0 rpy=0 0 0
- joint R_hip_roll_joint: axis -1 0 0 -> 1 0 0
- joint R_shoulder_pitch_joint: origin xyz=-0.015 0.2 0.3625 rpy=0 0 0 -> xyz=-0.015 -0.2 0.3625 rpy=0 0 0
- joint R_shoulder_roll_joint: axis -1 0 0 -> 1 0 0

File: pygmalion_locomotion/assets/pygmalion_v2/pygmalion_v4_printed_loop.urdf (robot description, URDF)
Before this commit: robot pygmalion_v4_printed_loop, 30 links, 29 joints
Links:
- link L_arm_link: geometry collision mesh filename=meshes/R_arm_hull.stl; visual mesh filename=meshes/R_arm.stl
- link L_crank_A: geometry visual mesh filename=meshes/R_crank_A.stl
- link L_crank_B: geometry visual mesh filename=meshes/R_crank_B.stl
- link L_foot_link: geometry collision mesh filename=meshes/R_foot_hull.stl; visual mesh filename=meshes/R_foot.stl
- link L_hip_pitch_link: geometry collision mesh filename=meshes/R_hip_pitch_link_hull.stl; visual mesh filename=meshes/R_hip_pitch_link.stl
- link L_hip_roll_link: geometry collision mesh filename=meshes/R_hip_roll_link_hull.stl; visual mesh filename=meshes/R_hip_roll_link.stl
- link L_rod_A: geometry visual mesh filename=meshes/R_rod_A.stl
- link L_rod_B: geometry visual mesh filename=meshes/R_rod_B.stl
- link L_shin_link: geometry collision mesh filename=meshes/R_shin_hull.stl; visual mesh filename=meshes/R_shin.stl
- link L_shoulder_pitch_link: geometry collision mesh filename=meshes/R_shoulder_pitch_link_hull.stl; visual mesh filename=meshes/R_shoulder_pitch_link.stl
- link L_thigh_link: geometry collision mesh filename=meshes/R_thigh_hull.stl; visual mesh filename=meshes/R_thigh.stl
- link R_arm_link: geometry collision mesh filename=meshes/arm_hull.stl; visual mesh filename=meshes/arm.stl
- link R_crank_A: geometry visual mesh filename=meshes/crank_A.stl
- link R_crank_B: geometry visual mesh filename=meshes/crank_B.stl
- link R_foot_link: geometry collision mesh filename=meshes/foot_hull.stl; visual mesh filename=meshes/foot.stl
- link R_hip_pitch_link: geometry collision mesh filename=meshes/hip_pitch_link_hull.stl; visual mesh filename=meshes/hip_pitch_link.stl
- link R_hip_roll_link: geometry collision mesh filename=meshes/hip_roll_link_hull.stl; visual mesh filename=meshes/hip_roll_link.stl
- link R_rod_A: geometry visual mesh filename=meshes/rod_A.stl
- link R_rod_B: geometry visual mesh filename=meshes/rod_B.stl
- link R_shin_link: geometry collision mesh filename=meshes/shin_hull.stl; visual mesh filename=meshes/shin.stl
- link R_shoulder_pitch_link: geometry collision mesh filename=meshes/shoulder_pitch_link_hull.stl; visual mesh filename=meshes/shoulder_pitch_link.stl
- link R_thigh_link: geometry collision mesh filename=meshes/thigh_hull.stl; visual mesh filename=meshes/thigh.stl
Joints:
- joint L_ankle_roll_joint: axis -1 0 0 -> 1 0 0
- joint L_crank_A_joint: origin xyz=-0.029945 -0.001718 -0.190034 rpy=0 0 0 -> xyz=-0.029945 0.001718 -0.190034 rpy=0 0 0
- joint L_crank_B_joint: origin xyz=-0.030055 0.001717 -0.290034 rpy=0 0 0 -> xyz=-0.030055 -0.001717 -0.290034 rpy=0 0 0
- joint L_hip_pitch_joint: origin xyz=0 -0.1237 0 rpy=0 0 0 -> xyz=0 0.1237 0 rpy=0 0 0
- joint L_hip_roll_joint: axis 1 0 0 -> -1 0 0
- joint L_rod_A_u1: origin xyz=-0.061494 0.042718 -0.021185 rpy=0 0 0 -> xyz=-0.061494 -0.042718 -0.021185 rpy=0 0 0
- joint L_rod_B_u1: origin xyz=-0.060039 -0.042717 -0.01522 rpy=0 0 0 -> xyz=-0.060039 0.042717 -0.01522 rpy=0 0 0
- joint L_shoulder_pitch_joint: origin xyz=-0.015 -0.2 0.3625 rpy=0 0 0 -> xyz=-0.015 0.2 0.3625 rpy=0 0 0
- joint L_shoulder_roll_joint: axis 1 0 0 -> -1 0 0
- joint R_ankle_roll_joint: axis 1 0 0 -> -1 0 0
- joint R_crank_A_joint: origin xyz=-0.029945 0.001718 -0.190034 rpy=0 0 0 -> xyz=-0.029945 -0.001718 -0.190034 rpy=0 0 0
- joint R_crank_B_joint: origin xyz=-0.030055 -0.001717 -0.290034 rpy=0 0 0 -> xyz=-0.030055 0.001717 -0.290034 rpy=0 0 0
- joint R_hip_pitch_joint: origin xyz=0 0.1237 0 rpy=0 0 0 -> xyz=0 -0.1237 0 rpy=0 0 0
- joint R_hip_roll_joint: axis -1 0 0 -> 1 0 0
- joint R_rod_A_u1: origin xyz=-0.061494 -0.042718 -0.021185 rpy=0 0 0 -> xyz=-0.061494 0.042718 -0.021185 rpy=0 0 0
- joint R_rod_B_u1: origin xyz=-0.060039 0.042717 -0.01522 rpy=0 0 0 -> xyz=-0.060039 -0.042717 -0.01522 rpy=0 0 0
- joint R_shoulder_pitch_joint: origin xyz=-0.015 0.2 0.3625 rpy=0 0 0 -> xyz=-0.015 -0.2 0.3625 rpy=0 0 0
- joint R_shoulder_roll_joint: axis -1 0 0 -> 1 0 0
